Commit message: Update resources

File: robots/iit/iCub/iCub_only_primitives.urdf (robot description, URDF)
Before this commit: robot iCub, 105 links, 104 joints
Joints:
- joint l_elbow: axis -8.811822027610106e-08 1.0 -2.2930406373689038e-07 -> 0.0 -1.0 0.0
- joint r_elbow: axis 2.494957698218059e-07 1.0 -2.454089553793892e-07 -> 0.0 -1.0 0.0
- joint r_shoulder_pitch: axis 1.4990443730766856e-07 1.0 -1.456618718975733e-07 -> 0.0 -1.0 0.0
- joint r_wrist_yaw: axis -2.494957698218059e-07 1.0 2.454089553793892e-07 -> 0.0 -1.0 0.0
