Commit message: Update iCub scenario

File: robots/iit/iCub/iCub.urdf (robot description, URDF)
Before this commit: robot iCub, 105 links, 104 joints
Joints:
- joint r_hand_middle_0_joint: limit lower=0.0 upper=0.0 effort=50000.0 velocity=50000.0 -> lower=0.0 upper=0.3490658503988659 effort=50000.0 velocity=50000.0

Commit message: Update demo

File: robots/iit/iCub/iCub.urdf (robot description, URDF)
Before this commit: robot iCub, 105 links, 104 joints
Joints:
- joint r_shoulder_pitch: limit lower=-3.054326295852661 upper=0.3490658402442932 effort=50000.0 velocity=120.0 -> lower=-0.3490658402442932 upper=3.054326295852661 effort=50000.0 velocity=120.0

Commit message: Fix iCub

File: robots/iit/iCub/iCub.urdf (robot description, URDF)
Before this commit: robot iCub, 105 links, 104 joints
Joints:
- joint r_shoulder_pitch: axis 1.4990443730766856e-07 1.0 -1.2401537219375314e-07 -> 1.4990443730766856e-07 -1.0 -1.2401537219375314e-07

Commit message: Update demo

File: robots/iit/iCub/iCub.urdf (robot description, URDF)
Before this commit: robot iCub, 105 links, 104 joints
Joints:
- joint l_gripper_tool_frame_joint: origin xyz=0.0 0.0 0.13 rpy=0.0 0.0 0.0 -> xyz=0.075 0.0 0.0 rpy=0.0 0.0 0.0
- joint r_gripper_tool_frame_joint: origin xyz=0.0 0.0 0.13 rpy=0.0 0.0 0.0 -> xyz=-0.075 0.0 0.0 rpy=0.0 0.0 0.0
- joint r_wrist_yaw: axis -2.4949582666522474e-07 -1.000000238418579 -2.7942487434984287e-08 -> -2.4949582666522474e-07 1.000000238418579 -2.7942487434984287e-08
