Commit message: Update robots

File: robots/unitree/urdf/g1/g1_29dof.urdf (robot description, URDF)
Before this commit: robot g1_29dof, 40 links, 39 joints
Links:
- removed link left_rubber_hand
- removed link right_rubber_hand
Joints:
- removed joint left_hand_palm_joint
- removed joint right_hand_palm_joint
