Commit message: Update demo

File: objects/montessori_toys/montessori_box/urdf/montessori_box.urdf (robot description, URDF)
Before this commit: robot montessori_box, 7 links, 6 joints
Links:
- link montessori_box: mass 6.423900127410889 -> 1.0220392942428589
- link montessori_drawer_1: mass 0.16877292096614838 -> 0.13218805193901062
- link montessori_drawer_1_handle: mass 0.004546803887933493 -> 0.005739745683968067
- link montessori_drawer_2: mass 0.16877292096614838 -> 0.13218805193901062
- link montessori_drawer_2_handle: mass 0.004546803887933493 -> 0.005739745683968067
- link montessori_drawer_3: mass 0.16877292096614838 -> 0.13218805193901062
- link montessori_drawer_3_handle: mass 0.004546803887933493 -> 0.005739745683968067
Joints:
- joint montessori_drawer_1_handle_joint: origin xyz=-0.07 0.0 0.0 rpy=0.0 0.0 0.0 -> xyz=-0.061 0.0 0.001 rpy=0.0 0.0 0.0
- joint montessori_drawer_1_joint: origin xyz=-0.004999999888241291 0.08929800242185593 0.0 rpy=0.0 0.0 0.0 -> xyz=-0.003000000026077032 0.08699999749660492 0.0 rpy=0.0 0.0 0.0
- joint montessori_drawer_2_handle_joint: origin xyz=-0.07 0.0 0.0 rpy=0.0 0.0 0.0 -> xyz=-0.061 0.0 0.001 rpy=0.0 0.0 0.0
- joint montessori_drawer_2_joint: origin xyz=-0.004999999888241291 0.0 0.0 rpy=0.0 0.0 0.0 -> xyz=-0.003000000026077032 0.0 0.0 rpy=0.0 0.0 0.0
- joint montessori_drawer_3_handle_joint: origin xyz=-0.07 0.0 0.0 rpy=0.0 0.0 0.0 -> xyz=-0.061 0.0 0.001 rpy=0.0 0.0 0.0
- joint montessori_drawer_3_joint: origin xyz=-0.004999999888241291 -0.08929800242185593 0.0 rpy=0.0 0.0 0.0 -> xyz=-0.003000000026077032 -0.08699999749660492 0.0 rpy=0.0 0.0 0.0

File: objects/montessori_toys/montessori_box/urdf/montessori_object_1.urdf (robot description, URDF)
Before this commit: robot montessori_object_1, 1 links, 0 joints
Links:
- link montessori_object_1: mass 0.004115183837711811 -> 0.0060821231454610825; geometry visual cylinder length=0.004000000189989805 radius=0.02199999988079071

File: objects/montessori_toys/montessori_box/urdf/montessori_object_2.urdf (robot description, URDF)
Before this commit: robot montessori_object_2, 1 links, 0 joints
Links:
- link montessori_object_2: mass 0.01134409662336111 -> 0.0213395357131958

File: objects/montessori_toys/montessori_box/urdf/montessori_object_3.urdf (robot description, URDF)
Before this commit: robot montessori_object_3, 1 links, 0 joints
Links:
- link montessori_object_3: mass 0.007762392051517963 -> 0.027000000700354576; geometry visual box size=0.029999999329447746 0.029999999329447746 0.029999999329447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

File: objects/montessori_toys/montessori_box/urdf/montessori_object_4.urdf (robot description, URDF)
Before this commit: robot montessori_object_4, 1 links, 0 joints
Links:
- link montessori_object_4: mass 0.013717278838157654 -> 0.033510319888591766; geometry visual sphere radius=0.019999999552965164

File: objects/montessori_toys/montessori_box/urdf/montessori_object_5.urdf (robot description, URDF)
Before this commit: robot montessori_object_5, 1 links, 0 joints
Links:
- link montessori_object_5: mass 0.008732691407203674 -> 0.024000000208616257; geometry visual box size=0.019999999552965164 0.03999999910593033 0.0299999993294477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

File: objects/montessori_toys/montessori_box/urdf/montessori_object_6.urdf (robot description, URDF)
Before this commit: robot montessori_object_6, 1 links, 0 joints
Links:
- link montessori_object_6: mass 0.006096568424254656 -> 0.021205751225352287; geometry visual cylinder length=0.029999999329447746 radius=0.014999999664723873

Commit message: Add holes

File: objects/montessori_toys/montessori_box/urdf/montessori_box.urdf (robot description, URDF)
Before this commit: robot montessori_box, 7 links, 6 joints
Links:
- added link montessori_hole_1
- added link montessori_hole_2
- added link montessori_hole_3
- added link montessori_hole_4
- added link montessori_hole_5
- added link montessori_hole_6
Joints:
- added joint montessori_hole_1_joint: type fixed, parent montessori_toys, child montessori_hole_1, origin xyz=0.025 0.091 0.04 rpy=0.0 0.0 0.0
- added joint montessori_hole_2_joint: type fixed, parent montessori_toys, child montessori_hole_2, origin xyz=0.0185 0 0.04 rpy=0.0 0.0 0.0
- added joint montessori_hole_3_joint: type fixed, parent montessori_toys, child montessori_hole_3, origin xyz=0.0205 -0.087 0.04 rpy=0.0 0.0 0.0
- added joint montessori_hole_4_joint: type fixed, parent montessori_toys, child montessori_hole_4, origin xyz=-0.0175 0.091 0.04 rpy=0.0 0.0 0.0
- added joint montessori_hole_5_joint: type fixed, parent montessori_toys, child montessori_hole_5, origin xyz=-0.0265 0 0.04 rpy=0.0 0.0 0.0
- added joint montessori_hole_6_joint: type fixed, parent montessori_toys, child montessori_hole_6, origin xyz=-0.0215 -0.087 0.04 rpy=0.0 0.0 0.0

Commit message: Update demo

File: objects/montessori_toys/montessori_box/urdf/montessori_box.urdf (robot description, URDF)
Before this commit: robot montessori_box, 13 links, 12 joints
Joints:
- joint montessori_hole_1_joint: parent montessori_toys -> montessori_box
- joint montessori_hole_2_joint: parent montessori_toys -> montessori_box
- joint montessori_hole_3_joint: parent montessori_toys -> montessori_box
- joint montessori_hole_4_joint: parent montessori_toys -> montessori_box
- joint montessori_hole_5_joint: parent montessori_toys -> montessori_box
- joint montessori_hole_6_joint: parent montessori_toys -> montessori_box
