Commit message: Fix demo

File: robots/shadow_hand/urdf/left_hand.urdf (robot description, URDF)
Before this commit: robot left_shadow_hand, 25 links, 24 joints
Links:
- link lh_palm_ref: geometry visual mesh filename=file://assets/stl/l_palm.stl scale=1.0 1.0 1.0

File: robots/shadow_hand/urdf/right_hand.urdf (robot description, URDF)
Before this commit: robot right_shadow_hand, 24 links, 23 joints
Links:
- link rh_palm: geometry collision box size=0.017999999225139618 0.024000000208616257 0.004000000189989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; collision box size=0.019999999552965164 0.024000000208616257 0.039999999105930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

Commit message: Add shadow_hand usd

File: robots/shadow_hand/urdf/left_hand.urdf (robot description, URDF)
Before this commit: robot left_shadow_hand, 25 links, 24 joints
Links:
- removed link lh_palm_ref
- removed link world
Joints:
- removed joint lh_palm_joint
- removed joint lh_palm_ref_joint

File: robots/shadow_hand/urdf/right_hand.urdf (robot description, URDF)
Before this commit: robot right_shadow_hand, 24 links, 23 joints
Links:
- removed link rh_palm_ref
Joints:
- removed joint rh_palm_ref_joint
